Commit message: urdf upload

File: urdf/panda.urdf (robot description, URDF)
Before this commit: robot panda, 12 links, 11 joints
Links:
- removed link panda_hand
- removed link panda_leftfinger
- removed link panda_rightfinger
- added link world
- link panda_link0: mass None -> 3.06; geometry collision mesh filename=package://franka_description/meshes/collision/link0.stl; visual mesh filename=package://franka_description/meshes/visual/link0.dae
- link panda_link1: mass None -> 2.34; geometry collision mesh filename=package://franka_description/meshes/collision/link1.stl; visual mesh filename=package://franka_description/meshes/visual/link1.dae
- link panda_link2: mass None -> 2.36; geometry collision cylinder length=0.12 radius=0.09; collision sphere radius=0.09
- link panda_link3: mass None -> 2.38; geometry collision cylinder length=0.15 radius=0.09; collision sphere radius=0.09
- link panda_link4: mass None -> 2.43; geometry collision cylinder length=0.12 radius=0.09; collision sphere radius=0.09
- link panda_link5: mass None -> 3.5; geometry collision cylinder length=0.1 radius=0.09; collision cylinder length=0.14 radius=0.055
- link panda_link6: mass None -> 1.47; geometry collision cylinder length=0.08 radius=0.08; collision sphere radius=0.08
- link panda_link7: mass None -> 0.45; geometry collision cylinder length=0.14 radius=0.07; collision sphere radius=0.07
- link panda_link8: mass None -> 0.45
Joints:
- removed joint panda_finger_joint1
- removed joint panda_finger_joint2
- removed joint panda_hand_joint
- joint panda_joint1: limit lower=-2.9671 upper=2.9671 effort=87 velocity=2.3925 -> lower=-2.8973 upper=2.8973 effort=87 velocity=2.1750
- joint panda_joint2: limit lower=-1.8326 upper=1.8326 effort=87 velocity=2.3925 -> lower=-1.7628 upper=1.7628 effort=87 velocity=2.1750
- joint panda_joint3: limit lower=-2.9671 upper=2.9671 effort=87 velocity=2.3925 -> lower=-2.8973 upper=2.8973 effort=87 velocity=2.1750
- joint panda_joint4: limit lower=-3.1416 upper=0.0873 effort=87 velocity=2.3925 -> lower=-3.0718 upper=-0.0698 effort=87 velocity=2.1750
- joint panda_joint5: limit lower=-2.9671 upper=2.9671 effort=12 velocity=2.8710 -> lower=-2.8973 upper=2.8973 effort=12 velocity=2.6100
- joint panda_joint6: limit lower=-0.0873 upper=3.8223 effort=12 velocity=2.8710 -> lower=-0.0175 upper=3.7525 effort=12 velocity=2.6100
- joint panda_joint7: limit lower=-2.9671 upper=2.9671 effort=12 velocity=2.8710 -> lower=-2.8973 upper=2.8973 effort=12 velocity=2.6100
- joint panda_joint8: axis 0 0 0 -> (none)
