Commit message: examples updated

File: examples/urdf/rrbot.urdf (robot description, URDF)
Before this commit: robot rrbot, 3 links, 2 joints
Links:
- added link ee, mass 0; collision box size=0.1 0.1 0.05; visual box size=0.1 0.1 0.05
- added link world
Joints:
- added joint fixed: type fixed, parent world, child link1
- added joint joint3: type fixed, parent link3, child ee, origin xyz=0 0 0.975 rpy=0 0 0
- joint joint1: limit (none) -> effort=100 velocity=10; origin xyz=0 0.1 1.95 rpy=0 0 0 -> xyz=0.0 0.1 1.95 rpy=0 3.14 0
- joint joint2: limit (none) -> effort=100 velocity=10
