Commit message: fix example bugs

File: examples/urdf/simplecube.urdf (robot description, URDF)
Before this commit: robot simpleCube, 3 links, 2 joints
Links:
- removed link Link1
- added link link, mass 0.20; collision mesh filename=package://simplecube_description/meshes/onedof/demoshaft.stl; visual mesh filename=package://simplecube_description/meshes/onedof/dae/demoshaf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
Joints:
- removed joint J1
- added joint joint: type revolute, parent cube_base, child link, origin xyz=0 0 0.033 rpy=0 0 0, axis 0 0 1, limit lower=-3.14 upper=3.14 effort=300 velocity=100
- joint dummy_base: type floating -> fixed
